File: Eagle/TI TS5Axx.brd (EAGLE design)
At the start: 38.5 x 36.1 mm, 31 parts, among them IC1 TS5A23159RSER, IC2 TS5A23159RSER, IC3 TS5A23159RSER, IC4 TS5A23159RSER, Q1 8Mhz, U1 LM1117MPX-1.8

Commit message: add alternative scheme
Routing:
- net GND: track 147.7 -> 177.4 mm, vias 8 -> 11
Changed lines of the file:
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@@
 <setting verticaltext="up"/>
 </settings>
-<grid distance="10" unitdist="mil" unit="mil" style="lines" multiple="1" display="yes" altdistance="5" altunitdist="mil" altunit="mil"/>
+<grid distance="20" unitdist="mil" unit="mil" style="lines" multiple="1" display="yes" altdistance="5" altunitdist="mil" altunit="mil"/>
 <layers>
 <layer number="1" name="Top" color="4" fill="1" visible="yes" active="yes"/>
@@
 <wire x1="59.36" y1="37.582" x2="20.828" y2="37.582" width="0" layer="20"/>
 <wire x1="20.828" y1="37.582" x2="20.828" y2="1.524" width="0" layer="20"/>
+<hole x="57.912" y="3.048" drill="0.508"/>
+<hole x="57.912" y="36.068" drill="0.508"/>
+<hole x="25.908" y="36.068" drill="0.508"/>
+<hole x="25.908" y="3.048" drill="0.508"/>
 </plain>
 <attributes>
@@
 </class>
 </classes>
-<designrules name="default">
+<designrules name="default *">
 <description language="de">&lt;b&gt;EAGLE Design Rules&lt;/b&gt;
 &lt;p&gt;
@@
 <param name="mtCopper" value="0.035mm 0.035mm 0.035mm 0.035mm 0.035mm 0.035mm 0.035mm 0.035mm 0.035mm 0.035mm 0.035mm 0.035mm 0.035mm 0.035mm 0.035mm 0.035mm"/>
 <param name="mtIsolate" value="1.5mm 0.15mm 0.2mm 0.15mm 0.2mm 0.15mm 0.2mm 0.15mm 0.2mm 0.15mm 0.2mm 0.15mm 0.2mm 0.15mm 0.2mm"/>
-<param name="mdWireWire" value="6mil"/>
-<param name="mdWirePad" value="6mil"/>
-<param name="mdWireVia" value="6mil"/>
+<param name="mdWireWire" value="3mil"/>
+<param name="mdWirePad" value="3mil"/>
+<param name="mdWireVia" value="3mil"/>
 <param name="mdPadPad" value="6mil"/>
-<param name="mdPadVia" value="6mil"/>
-<param name="mdViaVia" value="6mil"/>
-<param name="mdSmdPad" value="6mil"/>
-<param name="mdSmdVia" value="6mil"/>
-<param name="mdSmdSmd" value="6mil"/>
+<param name="mdPadVia" value="3mil"/>
+<param name="mdViaVia" value="3mil"/>
+<param name="mdSmdPad" value="3mil"/>
+<param name="mdSmdVia" value="3mil"/>
+<param name="mdSmdSmd" value="3mil"/>
 <param name="mdViaViaSameLayer" value="6mil"/>
 <param name="mnLayersViaInSmd" value="2"/>
 <param name="mdCopperDimension" value="40mil"/>
-<param name="mdDrill" value="6mil"/>
+<param name="mdDrill" value="3mil"/>
 <param name="mdSmdStop" value="0mil"/>
 <param name="msWidth" value="6mil"/>
-<param name="msDrill" value="0.35mm"/>
-<param name="msMicroVia" value="9.99mm"/>
-<param name="msBlindViaRatio" value="0.5"/>
+<param name="msDrill" value="0.01mm"/>
+<param name="msMicroVia" value="0.01mm"/>
+<param name="msBlindViaRatio" value="0.01"/>
 <param name="rvPadTop" value="0.25"/>
 <param name="rvPadInner" value="0.25"/>
@@
 <param name="mvCreamFrame" value="0"/>
 <param name="mlMinStopFrame" value="4mil"/>
-<param name="mlMaxStopFrame" value="4mil"/>
+<param name="mlMaxStopFrame" value="12mil"/>
 <param name="mlMinCreamFrame" value="0mil"/>
 <param name="mlMaxCreamFrame" value="0mil"/>
@@
 <wire x1="53.594" y1="17.526" x2="53.594" y2="10.16" width="0.6096" layer="16"/>
 <wire x1="53.594" y1="10.16" x2="51.816" y2="8.382" width="0.6096" layer="16"/>
-<wire x1="51.816" y1="8.382" x2="50.292" y2="8.382" width="0.6096" layer="16"/>
-<wire x1="50.292" y1="8.382" x2="43.434" y2="8.382" width="0.6096" layer="16"/>
 <wire x1="43.434" y1="8.382" x2="41.148" y2="10.668" width="0.6096" layer="16"/>
 <wire x1="52.832" y1="24.384" x2="52.832" y2="18.542" width="0.6096" layer="16"/>
 <via x="53.594" y="17.526" extent="1-16" drill="0.2" diameter="0.55" shape="square"/>
-<via x="50.292" y="8.382" extent="1-16" drill="0.2" diameter="0.55" shape="square"/>
 <via x="41.148" y="10.668" extent="1-16" drill="0.2" diameter="0.55" shape="square"/>
 <wire x1="41.148" y1="10.668" x2="42.462" y2="11.982" width="0.3048" layer="1"/>
 <wire x1="42.462" y1="11.982" x2="43.548" y2="11.982" width="0.3048" layer="1"/>
-<wire x1="50.248" y1="10.782" x2="50.248" y2="8.426" width="0.3048" layer="1"/>
-<wire x1="50.248" y1="8.426" x2="50.292" y2="8.382" width="0.3048" layer="1"/>
 <wire x1="51.448" y1="17.482" x2="53.55" y2="17.482" width="0.3048" layer="1"/>
 <wire x1="53.55" y1="17.482" x2="53.594" y2="17.526" width="0.3048" layer="1"/>
@@
 <wire x1="23.622" y1="6.35" x2="25.204" y2="6.35" width="0.3048" layer="1"/>
 <wire x1="25.204" y1="6.35" x2="25.208" y2="6.354" width="0.3048" layer="1"/>
+<wire x1="51.816" y1="8.382" x2="51.054" y2="8.382" width="0.6096" layer="16"/>
+<wire x1="51.054" y1="8.382" x2="43.434" y2="8.382" width="0.6096" layer="16"/>
+<wire x1="50.248" y1="9.79384375" x2="50.248" y2="10.782" width="0.3048" layer="1"/>
+<wire x1="50.646" y1="9.39584375" x2="50.646" y2="8.79" width="0.3048" layer="1"/>
+<wire x1="50.646" y1="9.39584375" x2="50.248" y2="9.79384375" width="0.3048" layer="1"/>
+<via x="51.054" y="8.382" extent="1-16" drill="0.2"/>
+<wire x1="50.646" y1="8.79" x2="51.054" y2="8.382" width="0.3048" layer="1"/>
 </signal>
 <signal name="GND">
@@
 <wire x1="52.832" y1="26.162" x2="50.154" y2="28.84" width="0.6096" layer="1"/>
 <wire x1="52.832" y1="20.828" x2="52.832" y2="26.162" width="0.6096" layer="1"/>
-<wire x1="51.448" y1="16.982" x2="53.10055" y2="16.982" width="0.3048" layer="1"/>
+<wire x1="51.448" y1="16.982" x2="52.578" y2="16.982" width="0.3048" layer="1"/>
+<wire x1="52.578" y1="16.982" x2="53.10055" y2="16.982" width="0.3048" layer="1"/>
 <wire x1="53.10055" y1="16.982" x2="53.16455" y2="16.918" width="0.3048" layer="1"/>
 <wire x1="53.16455" y1="16.918" x2="54.51" y2="16.918" width="0.3048" layer="1"/>
@@
 <wire x1="41.656" y1="23.368" x2="41.148" y2="22.86" width="0.8128" layer="1"/>
 <wire x1="41.148" y1="22.86" x2="40.386" y2="22.86" width="0.8128" layer="1"/>
-<via x="40.386" y="22.86" extent="1-16" drill="0.35" diameter="0.1778"/>
+<via x="40.386" y="22.86" extent="1-16" drill="0.35"/>
 <wire x1="40.386" y1="22.86" x2="40.386" y2="26.924" width="0.8128" layer="16"/>
 <via x="40.386" y="26.924" extent="1-16" drill="0.35" diameter="0.1778"/>
@@
 <vertex x="20.828" y="1.524"/>
 </polygon>
-<wire x1="51.448" y1="16.982" x2="46.748" y2="18.682" width="0" layer="19" extent="1-1"/>
-<wire x1="49.748" y1="10.782" x2="51.448" y2="16.982" width="0" layer="19" extent="1-1"/>
-<wire x1="43.548" y1="12.482" x2="49.748" y2="10.782" width="0" layer="19" extent="1-1"/>
+<wire x1="52.578" y1="16.982" x2="52.578" y2="16.51" width="0.1524" layer="1"/>
+<via x="52.578" y="16.51" extent="1-16" drill="0.2"/>
+<wire x1="52.578" y1="10.414" x2="51.308" y2="9.144" width="0.6096" layer="16"/>
+<wire x1="51.308" y1="9.144" x2="50.038" y2="9.144" width="0.6096" layer="16"/>
+<wire x1="50.038" y1="9.144" x2="43.942" y2="9.144" width="0.6096" layer="16"/>
+<wire x1="43.942" y1="9.144" x2="41.148" y2="11.938" width="0.6096" layer="16"/>
+<wire x1="52.578" y1="16.51" x2="52.578" y2="10.414" width="0.6096" layer="16"/>
+<via x="41.148" y="11.938" extent="1-16" drill="0.1778"/>
+<wire x1="41.148" y1="11.938" x2="41.692" y2="12.482" width="0.3048" layer="1"/>
+<wire x1="41.692" y1="12.482" x2="43.548" y2="12.482" width="0.3048" layer="1"/>
+<via x="50.038" y="9.144" extent="1-16" drill="0.2032"/>
+<wire x1="50.038" y1="9.144" x2="49.748" y2="9.434" width="0.3048" layer="1"/>
+<wire x1="49.748" y1="9.434" x2="49.748" y2="10.782" width="0.3048" layer="1"/>
+<wire x1="46.7908" y1="18.6392" x2="46.748" y2="18.682" width="0.3048" layer="1"/>
+<wire x1="47.91695" y1="16.982" x2="46.7908" y2="18.10815" width="0.3048" layer="1"/>
+<wire x1="46.7908" y1="18.10815" x2="46.7908" y2="18.6392" width="0.3048" layer="1"/>
+<wire x1="51.448" y1="16.982" x2="47.91695" y2="16.982" width="0.3048" layer="1"/>
 </signal>
 <signal name="VDD">
@@
 <via x="51.816" y="29.21" extent="1-16" drill="0.2" diameter="0.55"/>
 <wire x1="51.816" y1="29.21" x2="51.816" y2="26.416" width="0.6096" layer="16"/>
+<wire x1="51.816" y1="26.416" x2="46.228" y2="20.828" width="0.6096" layer="16"/>
 <wire x1="46.228" y1="20.828" x2="46.228" y2="20.32" width="0.6096" layer="16"/>
-<wire x1="51.816" y1="26.416" x2="46.228" y2="20.828" width="0.6096" layer="16"/>
-<via x="46.228" y="20.32" extent="1-16" drill="0.2" diameter="0.55"/>
-<wire x1="46.228" y1="20.32" x2="46.248" y2="20.3" width="0.3048" layer="1"/>
-<wire x1="46.248" y1="20.3" x2="46.248" y2="18.682" width="0.3048" layer="1"/>
+<via x="46.228" y="20.32" extent="1-16" drill="0.2"/>
+<wire x1="46.228" y1="20.32" x2="46.228" y2="19.95058125" width="0.3048" layer="1"/>
+<wire x1="46.228" y1="19.95058125" x2="46.248" y2="19.93058125" width="0.3048" layer="1"/>
+<wire x1="46.248" y1="19.93058125" x2="46.248" y2="18.682" width="0.3048" layer="1"/>
 </signal>
 <signal name="N$1">
@@
 <wire x1="25.4" y1="27.432" x2="25.4" y2="25.654" width="0.3048" layer="1"/>
 <wire x1="25.4" y1="25.654" x2="24.384" y2="24.638" width="0.3048" layer="1"/>
-<via x="24.384" y="24.638" extent="1-16" drill="0.1016" diameter="0.127"/>
+<via x="24.384" y="24.638" extent="1-16" drill="0.2"/>
 <wire x1="24.384" y1="24.638" x2="22.098" y2="22.352" width="0.3048" layer="16"/>
 <wire x1="25.908" y1="18.862" x2="25.908" y2="18.034" width="0.3048" layer="1"/>
@@
 <via x="32.258" y="18.796" extent="1-16" drill="0.127" diameter="0.1778"/>
 <wire x1="32.258" y1="18.796" x2="38.1" y2="18.796" width="0.3048" layer="16"/>
-<via x="38.1" y="18.796" extent="1-16" drill="0.127" diameter="0.1778"/>
+<via x="38.1" y="18.796" extent="1-16" drill="0.2"/>
 <wire x1="38.1" y1="18.796" x2="39.116" y2="18.796" width="0.3048" layer="1"/>
 <wire x1="39.116" y1="18.796" x2="40.64" y2="20.32" width="0.3048" layer="1"/>
@@
 <wire x1="27.686" y1="12.7" x2="28.702" y2="12.7" width="0.3048" layer="16"/>
 <wire x1="27.686" y1="9.906" x2="27.686" y2="12.7" width="0.3048" layer="16"/>
-<via x="27.686" y="12.7" extent="1-16" drill="0.127" diameter="0.1524"/>
+<via x="27.686" y="12.7" extent="1-16" drill="0.127"/>
 <wire x1="26.162" y1="12.7" x2="27.686" y2="12.7" width="0.3048" layer="1"/>
 <contactref element="U$1" pad="25"/>
